File: v00/v00_hardware/v00_hardware_hole.brd (EAGLE design)
At the start: 50.8 x 50.8 mm, 12 parts

Commit message: hardware changes
Parts:
- removed D1, D2, D3, D4: (no value), SparkFun-LED:LED_5MM
- added JP4, JP5, JP6, JP7: (no value), adafruit:1X01
- added LED1, LED2, LED3, LED4: (no value), adafruit:LED5MM
Connections:
- net GND: now also JP5.1, LED1.A, LED2.A, LED3.A, LED4.A; no longer D1.A, D2.A, D3.A, D4.A
- net N$1: now also LED1.K; no longer D1.K
- net N$2: now also LED2.K; no longer D2.K
- net N$3: now also LED3.K; no longer D3.K
- net N$4: now also LED4.K; no longer D4.K
- net N$7: now also JP6.1, JP7.1
- net VCC: now also JP4.1
Routing:
- net N$7: track 121.2 -> 141.2 mm
- net VCC: track 63.9 -> 70.8 mm
- net GND: track 181.4 -> 184.7 mm
- net N$8: track 44.9 -> 46.7 mm
Changed lines of the file:
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@@
 </autorouter>
 <elements>
-<element name="D1" library="SparkFun-LED" package="LED_5MM" value="" x="76.2" y="88.9"/>
-<element name="D2" library="SparkFun-LED" package="LED_5MM" value="" x="76.2" y="12.7"/>
-<element name="D3" library="SparkFun-LED" package="LED_5MM" value="" x="38.1" y="50.8" rot="R270"/>
-<element name="D4" library="SparkFun-LED" package="LED_5MM" value="" x="114.3" y="50.8" rot="R90"/>
 <element name="R1" library="adafruit" package="0204/7" value="" x="85.09" y="88.9" rot="R180"/>
 <element name="R2" library="adafruit" package="0204/7" value="" x="85.09" y="12.7" rot="R180"/>
@@
 <element name="JP2" library="pinhead" library_urn="urn:adsk.eagle:library:325" package="1X04" package3d_urn="urn:adsk.eagle:package:22407/2" value="" x="46.99" y="78.74" rot="R45"/>
 <element name="JP3" library="pinhead" library_urn="urn:adsk.eagle:library:325" package="1X04" package3d_urn="urn:adsk.eagle:package:22407/2" value="" x="52.968025" y="72.761975" rot="R45"/>
+<element name="JP4" library="adafruit" package="1X01" value="" x="54.61" y="86.36" rot="R45"/>
+<element name="JP5" library="adafruit" package="1X01" value="" x="57.521971875" y="82.921975" rot="R45"/>
+<element name="LED1" library="adafruit" package="LED5MM" value="" x="76.2" y="88.9"/>
+<element name="LED2" library="adafruit" package="LED5MM" value="" x="76.2" y="12.7"/>
+<element name="LED3" library="adafruit" package="LED5MM" value="" x="38.1" y="50.8" rot="R270"/>
+<element name="LED4" library="adafruit" package="LED5MM" value="" x="114.3" y="50.8" rot="R90"/>
+<element name="JP6" library="adafruit" package="1X01" value="" x="55.88" y="11.43"/>
+<element name="JP7" library="adafruit" package="1X01" value="" x="63.5" y="19.05"/>
 </elements>
 <signals>
-<signal name="N$1">
-<contactref element="D1" pad="K"/>
-<contactref element="R1" pad="2"/>
-<wire x1="77.47" y1="88.9" x2="81.28" y2="88.9" width="1" layer="16"/>
-</signal>
-<signal name="N$2">
-<contactref element="D2" pad="K"/>
-<contactref element="R2" pad="2"/>
-<wire x1="81.28" y1="12.7" x2="77.47" y2="12.7" width="1" layer="16"/>
-</signal>
-<signal name="N$3">
-<contactref element="D3" pad="K"/>
-<contactref element="R3" pad="2"/>
-<wire x1="38.1" y1="49.53" x2="38.1" y2="43.18" width="1" layer="16"/>
-</signal>
-<signal name="N$4">
-<contactref element="D4" pad="K"/>
-<contactref element="R4" pad="2"/>
-<wire x1="114.3" y1="52.07" x2="114.3" y2="55.88" width="1" layer="16"/>
-</signal>
 <signal name="N$7">
 <contactref element="R1" pad="1"/>
@@
 <wire x1="109.22" y1="40.64" x2="88.15400625" y2="19.57400625" width="1" layer="16"/>
 <wire x1="88.15400625" y1="19.57400625" x2="74.18689375" y2="19.57400625" width="1" layer="16"/>
-<wire x1="72.3928875" y1="17.78" x2="63.5" y2="17.78" width="1" layer="16"/>
-<wire x1="74.18689375" y1="19.57400625" x2="72.3928875" y2="17.78" width="1" layer="16"/>
+<wire x1="72.3928875" y1="17.78" x2="74.18689375" y2="19.57400625" width="1" layer="16"/>
 <wire x1="47.888025" y1="18.369871875" x2="46.99" y2="17.471846875" width="1" layer="16"/>
+<contactref element="JP6" pad="1"/>
+<contactref element="JP7" pad="1"/>
+<wire x1="46.99" y1="12.7" x2="49.53" y2="10.16" width="1" layer="16"/>
+<wire x1="54.61" y1="10.16" x2="55.88" y2="11.43" width="1" layer="16"/>
 <wire x1="46.99" y1="17.471846875" x2="46.99" y2="12.7" width="1" layer="16"/>
-<wire x1="46.99" y1="12.7" x2="48.26" y2="11.43" width="1" layer="16"/>
-<wire x1="47.888025" y1="18.369871875" x2="63.5" y2="17.78" width="0" layer="19" extent="16-16"/>
+<wire x1="49.53" y1="10.16" x2="54.61" y2="10.16" width="1" layer="16"/>
+<wire x1="63.5" y1="19.05" x2="64.77" y2="17.78" width="1" layer="16"/>
+<wire x1="64.77" y1="17.78" x2="72.3928875" y2="17.78" width="1" layer="16"/>
+<wire x1="55.88" y1="11.43" x2="63.5" y2="19.05" width="1" layer="1"/>
 </signal>
 <signal name="N$8">
@@
 <wire x1="49.684078125" y1="16.57381875" x2="49.684078125" y2="15.96119375" width="1" layer="16"/>
 <wire x1="49.684078125" y1="15.96119375" x2="49.373321875" y2="15.6504375" width="1" layer="16"/>
-<wire x1="49.373321875" y1="13.905103125" x2="53.118425" y2="10.16" width="1" layer="16"/>
-<wire x1="86.36" y1="10.16" x2="88.9" y2="12.7" width="1" layer="16"/>
-<wire x1="53.118425" y1="10.16" x2="86.36" y2="10.16" width="1" layer="16"/>
+<wire x1="49.373321875" y1="13.905103125" x2="50.6074625" y2="12.6709625" width="1" layer="16"/>
+<wire x1="50.6074625" y1="12.6709625" x2="53.3109625" y2="12.6709625" width="1" layer="16"/>
+<wire x1="53.3109625" y1="12.6709625" x2="55.88" y2="15.24" width="1" layer="16"/>
+<wire x1="55.88" y1="15.24" x2="56.27761875" y2="15.24" width="1" layer="16"/>
+<wire x1="82.1631875" y1="10.56779375" x2="84.29539375" y2="12.7" width="1" layer="16"/>
+<wire x1="84.29539375" y1="12.7" x2="88.9" y2="12.7" width="1" layer="16"/>
+<wire x1="56.27761875" y1="15.24" x2="60.949825" y2="10.56779375" width="1" layer="16"/>
+<wire x1="60.949825" y1="10.56779375" x2="82.1631875" y2="10.56779375" width="1" layer="16"/>
 </signal>
 <signal name="N$9">
@@
 </signal>
 <signal name="GND">
-<contactref element="D1" pad="A"/>
-<contactref element="D2" pad="A"/>
-<contactref element="D3" pad="A"/>
-<contactref element="D4" pad="A"/>
 <contactref element="U$1" pad="14"/>
 <wire x1="45.781215625" y1="30.018846875" x2="46.091975" y2="30.32960625" width="1" layer="16"/>
 <wire x1="46.091975" y1="30.32960625" x2="46.091975" y2="30.942228125" width="1" layer="16"/>
 <wire x1="45.781215625" y1="28.273515625" x2="45.781215625" y2="30.018846875" width="1" layer="16"/>
-<wire x1="74.93" y1="12.7" x2="61.35473125" y2="12.7" width="1" layer="16"/>
-<wire x1="61.35473125" y1="12.7" x2="45.781215625" y2="28.273515625" width="1" layer="16"/>
+<wire x1="45.781215625" y1="28.273515625" x2="61.35473125" y2="12.7" width="1" layer="16"/>
 <wire x1="40.33380625" y1="36.087775" x2="46.091975" y2="30.32960625" width="1" layer="16"/>
-<wire x1="75.23619375" y1="13.625275" x2="76.544725" y2="14.93380625" width="1" layer="16"/>
-<wire x1="74.93" y1="12.7" x2="75.23619375" y2="13.00619375" width="1" layer="16"/>
-<wire x1="75.23619375" y1="13.00619375" x2="75.23619375" y2="13.625275" width="1" layer="16"/>
-<wire x1="76.544725" y1="14.93380625" x2="91.13380625" y2="14.93380625" width="1" layer="16"/>
-<wire x1="114.3" y1="38.1" x2="114.3" y2="49.53" width="1" layer="16"/>
-<wire x1="91.13380625" y1="14.93380625" x2="114.3" y2="38.1" width="1" layer="16"/>
 <contactref element="JP3" pad="1"/>
 <contactref element="JP3" pad="4"/>
 <contactref element="JP3" pad="3"/>
 <contactref element="JP3" pad="2"/>
-<wire x1="38.1" y1="52.07" x2="38.1" y2="57.89395" width="1" layer="16"/>
 <wire x1="38.1" y1="57.89395" x2="50.273946875" y2="70.067896875" width="1" layer="16"/>
 <wire x1="50.273946875" y1="70.067896875" x2="52.069996875" y2="71.863946875" width="1" layer="16"/>
 <wire x1="53.86605" y1="73.66" x2="52.069996875" y2="71.863946875" width="1" layer="16"/>
 <wire x1="53.86605" y1="73.66" x2="55.6621" y2="75.45605" width="1" layer="16"/>
-<wire x1="55.6621" y1="75.45605" x2="69.10605" y2="88.9" width="1" layer="16"/>
+<wire x1="55.6621" y1="75.45605" x2="60.588025" y2="80.381975" width="1" layer="16"/>
+<wire x1="60.588025" y1="80.381975" x2="69.10605" y2="88.9" width="1" layer="16"/>
+<wire x1="40.33380625" y1="36.087775" x2="40.33380625" y2="51.10619375" width="1" layer="16"/>
+<contactref element="JP5" pad="1"/>
+<wire x1="57.521971875" y1="82.921975" x2="60.061971875" y2="80.381975" width="1" layer="16"/>
+<wire x1="60.061971875" y1="80.381975" x2="60.588025" y2="80.381975" width="1" layer="16"/>
+<contactref element="LED1" pad="A"/>
+<contactref element="LED2" pad="A"/>
+<contactref element="LED3" pad="A"/>
+<contactref element="LED4" pad="A"/>
+<wire x1="40.33380625" y1="51.10619375" x2="39.37" y2="52.07" width="1" layer="16"/>
+<wire x1="39.37" y1="52.07" x2="38.1" y2="52.07" width="1" layer="16"/>
+<wire x1="38.1" y1="57.89395" x2="38.1" y2="52.07" width="1" layer="16"/>
 <wire x1="69.10605" y1="88.9" x2="74.93" y2="88.9" width="1" layer="16"/>
-<wire x1="38.1" y1="52.07" x2="39.37" y2="52.07" width="1" layer="16"/>
-<wire x1="39.37" y1="52.07" x2="40.33380625" y2="51.10619375" width="1" layer="16"/>
-<wire x1="40.33380625" y1="51.10619375" x2="40.33380625" y2="36.087775" width="1" layer="16"/>
+<wire x1="61.35473125" y1="12.7" x2="74.93" y2="12.7" width="1" layer="16"/>
+<wire x1="74.93" y1="12.7" x2="75.33779375" y2="13.10779375" width="1" layer="16"/>
+<wire x1="75.33779375" y1="13.10779375" x2="75.33779375" y2="13.5831875" width="1" layer="16"/>
+<wire x1="75.33779375" y1="13.5831875" x2="77.7406" y2="15.98599375" width="1" layer="16"/>
+<wire x1="90.91599375" y1="15.98599375" x2="114.3" y2="39.37" width="1" layer="16"/>
+<wire x1="114.3" y1="39.37" x2="114.3" y2="49.53" width="1" layer="16"/>
+<wire x1="77.7406" y1="15.98599375" x2="90.91599375" y2="15.98599375" width="1" layer="16"/>
 </signal>
 <signal name="N$5">
@@
 <wire x1="44.295921875" y1="76.045921875" x2="35.56" y2="67.31" width="1" layer="16"/>
 <wire x1="35.56" y1="67.31" x2="35.56" y2="30.697896875" width="1" layer="16"/>
+<contactref element="JP4" pad="1"/>
+<wire x1="54.61" y1="86.36" x2="49.684075" y2="81.434075" width="1" layer="16"/>
+</signal>
+<signal name="N$1">
+<contactref element="R1" pad="2"/>
+<contactref element="LED1" pad="K"/>
+<wire x1="81.28" y1="88.9" x2="77.47" y2="88.9" width="1" layer="16"/>
+</signal>
+<signal name="N$2">
+<contactref element="R2" pad="2"/>
+<contactref element="LED2" pad="K"/>
+<wire x1="77.47" y1="12.7" x2="81.28" y2="12.7" width="1" layer="16"/>
+</signal>
+<signal name="N$3">
+<contactref element="R3" pad="2"/>
+<contactref element="LED3" pad="K"/>
+<wire x1="38.1" y1="49.53" x2="38.1" y2="43.18" width="1" layer="16"/>
+</signal>
+<signal name="N$4">
+<contactref element="R4" pad="2"/>
+<contactref element="LED4" pad="K"/>
+<wire x1="114.3" y1="52.07" x2="114.3" y2="55.88" width="1" layer="16"/>
 </signal>
 </signals>
