File: v00/v00_hardware/v00_hardware_hole.sch (EAGLE design)
At the start: 12 parts

Commit message: hardware changes
Parts:
- removed D1, D2, D3, D4: (no value), SparkFun-LED:LED5MM
- added JP4, JP5, JP6, JP7: (no value), adafruit:PINHD-1X1
- added LED1, LED2, LED3, LED4: (no value), adafruit:LED5MM
Connections:
- net GND: now also JP5.1, LED1.A, LED2.A, LED3.A, LED4.A; no longer D1.A, D2.A, D3.A, D4.A
- net N$1: now also LED1.C; no longer D1.C
- net N$2: now also LED2.C; no longer D2.C
- net N$3: now also LED3.C; no longer D3.C
- net N$4: now also LED4.C; no longer D4.C
- net N$7: now also JP6.1, JP7.1
- net VCC: now also JP4.1
Changed lines of the file:
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@@
 </classes>
 <parts>
-<part name="D1" library="SparkFun-LED" deviceset="LED" device="5MM"/>
 <part name="U$1" library="SparkFun-IC-Microcontroller" deviceset="ATTINY84" device="ATTINY84-20PU"/>
 <part name="R1" library="adafruit" deviceset="R-US_" device="0204/7"/>
-<part name="D2" library="SparkFun-LED" deviceset="LED" device="5MM"/>
-<part name="D3" library="SparkFun-LED" deviceset="LED" device="5MM"/>
-<part name="D4" library="SparkFun-LED" deviceset="LED" device="5MM"/>
 <part name="R2" library="adafruit" deviceset="R-US_" device="0204/7"/>
 <part name="R3" library="adafruit" deviceset="R-US_" device="0204/7"/>
@@
 <part name="JP2" library="pinhead" library_urn="urn:adsk.eagle:library:325" deviceset="PINHD-1X4" device="" package3d_urn="urn:adsk.eagle:package:22407/2"/>
 <part name="JP3" library="pinhead" library_urn="urn:adsk.eagle:library:325" deviceset="PINHD-1X4" device="" package3d_urn="urn:adsk.eagle:package:22407/2"/>
+<part name="JP4" library="adafruit" deviceset="PINHD-1X1" device=""/>
+<part name="JP5" library="adafruit" deviceset="PINHD-1X1" device=""/>
+<part name="SUPPLY3" library="SparkFun-PowerSymbols" deviceset="VCC" device=""/>
+<part name="GND5" library="SparkFun-PowerSymbols" deviceset="GND" device=""/>
+<part name="LED1" library="adafruit" deviceset="LED" device="5MM"/>
+<part name="LED2" library="adafruit" deviceset="LED" device="5MM"/>
+<part name="LED3" library="adafruit" deviceset="LED" device="5MM"/>
+<part name="LED4" library="adafruit" deviceset="LED" device="5MM"/>
+<part name="JP6" library="adafruit" deviceset="PINHD-1X1" device=""/>
+<part name="JP7" library="adafruit" deviceset="PINHD-1X1" device=""/>
 </parts>
 <sheets>
@@
 </plain>
 <instances>
-<instance part="D1" gate="G$1" x="182.88" y="78.74"/>
 <instance part="U$1" gate="G$1" x="101.6" y="48.26"/>
 <instance part="R1" gate="G$1" x="182.88" y="68.58" rot="R90"/>
-<instance part="D2" gate="G$1" x="190.5" y="78.74"/>
-<instance part="D3" gate="G$1" x="198.12" y="78.74"/>
-<instance part="D4" gate="G$1" x="205.74" y="78.74"/>
 <instance part="R2" gate="G$1" x="190.5" y="68.58" rot="R90"/>
 <instance part="R3" gate="G$1" x="198.12" y="68.58" rot="R90"/>
@@
 <instance part="JP2" gate="A" x="-15.24" y="96.52"/>
 <instance part="JP3" gate="A" x="-15.24" y="76.2"/>
+<instance part="JP4" gate="G$1" x="30.48" y="96.52"/>
+<instance part="JP5" gate="G$1" x="30.48" y="78.74"/>
+<instance part="SUPPLY3" gate="G$1" x="20.32" y="96.52"/>
+<instance part="GND5" gate="1" x="20.32" y="81.28" rot="R180"/>
+<instance part="LED1" gate="G$1" x="182.88" y="78.74"/>
+<instance part="LED2" gate="G$1" x="190.5" y="78.74"/>
+<instance part="LED3" gate="G$1" x="198.12" y="78.74"/>
+<instance part="LED4" gate="G$1" x="205.74" y="78.74"/>
+<instance part="JP6" gate="G$1" x="149.86" y="71.12"/>
+<instance part="JP7" gate="G$1" x="162.56" y="71.12"/>
 </instances>
 <busses>
 </busses>
 <nets>
-<net name="N$1" class="0">
-<segment>
-<pinref part="D1" gate="G$1" pin="C"/>
-<pinref part="R1" gate="G$1" pin="2"/>
-</segment>
-</net>
-<net name="N$2" class="0">
-<segment>
-<pinref part="D2" gate="G$1" pin="C"/>
-<pinref part="R2" gate="G$1" pin="2"/>
-</segment>
-</net>
-<net name="N$3" class="0">
-<segment>
-<pinref part="D3" gate="G$1" pin="C"/>
-<pinref part="R3" gate="G$1" pin="2"/>
-</segment>
-</net>
-<net name="N$4" class="0">
-<segment>
-<pinref part="D4" gate="G$1" pin="C"/>
-<pinref part="R4" gate="G$1" pin="2"/>
-</segment>
-</net>
 <net name="N$7" class="0">
 <segment>
@@
 <wire x1="182.88" y1="60.96" x2="182.88" y2="63.5" width="0.1524" layer="91"/>
 <pinref part="U$1" gate="G$1" pin="(PCINT10/INT0/OC0A/CKOUT)PB2"/>
-<wire x1="182.88" y1="60.96" x2="127" y2="60.96" width="0.1524" layer="91"/>
+<wire x1="182.88" y1="60.96" x2="160.02" y2="60.96" width="0.1524" layer="91"/>
+<pinref part="JP6" gate="G$1" pin="1"/>
+<wire x1="160.02" y1="60.96" x2="147.32" y2="60.96" width="0.1524" layer="91"/>
+<wire x1="147.32" y1="60.96" x2="127" y2="60.96" width="0.1524" layer="91"/>
+<wire x1="147.32" y1="71.12" x2="147.32" y2="60.96" width="0.1524" layer="91"/>
+<pinref part="JP7" gate="G$1" pin="1"/>
+<wire x1="160.02" y1="71.12" x2="160.02" y2="60.96" width="0.1524" layer="91"/>
 </segment>
 </net>
@@
 </net>
 <net name="GND" class="0">
-<segment>
-<pinref part="D1" gate="G$1" pin="A"/>
-<pinref part="GND1" gate="1" pin="GND"/>
-</segment>
-<segment>
-<pinref part="D2" gate="G$1" pin="A"/>
-<pinref part="GND2" gate="1" pin="GND"/>
-</segment>
-<segment>
-<pinref part="D3" gate="G$1" pin="A"/>
-<pinref part="GND3" gate="1" pin="GND"/>
-</segment>
-<segment>
-<pinref part="D4" gate="G$1" pin="A"/>
-<pinref part="GND4" gate="1" pin="GND"/>
-</segment>
 <segment>
 <pinref part="U$1" gate="G$1" pin="GND"/>
@@
 <wire x1="-17.78" y1="78.74" x2="-10.16" y2="78.74" width="0.1524" layer="91"/>
 </segment>
+<segment>
+<pinref part="JP5" gate="G$1" pin="1"/>
+<pinref part="GND5" gate="1" pin="GND"/>
+<wire x1="20.32" y1="78.74" x2="27.94" y2="78.74" width="0.1524" layer="91"/>
+</segment>
+<segment>
+<pinref part="GND1" gate="1" pin="GND"/>
+<pinref part="LED1" gate="G$1" pin="A"/>
+</segment>
+<segment>
+<pinref part="GND2" gate="1" pin="GND"/>
+<pinref part="LED2" gate="G$1" pin="A"/>
+</segment>
+<segment>
+<pinref part="GND3" gate="1" pin="GND"/>
+<pinref part="LED3" gate="G$1" pin="A"/>
+</segment>
+<segment>
+<pinref part="GND4" gate="1" pin="GND"/>
+<pinref part="LED4" gate="G$1" pin="A"/>
+</segment>
 </net>
 <net name="VCC" class="0">
@@
 <wire x1="-10.16" y1="101.6" x2="-17.78" y2="101.6" width="0.1524" layer="91"/>
 </segment>
+<segment>
+<pinref part="JP4" gate="G$1" pin="1"/>
+<pinref part="SUPPLY3" gate="G$1" pin="VCC"/>
+<wire x1="20.32" y1="96.52" x2="27.94" y2="96.52" width="0.1524" layer="91"/>
+</segment>
 </net>
 <net name="N$5" class="0">
@@
 </segment>
 </net>
+<net name="N$1" class="0">
+<segment>
+<pinref part="R1" gate="G$1" pin="2"/>
+<pinref part="LED1" gate="G$1" pin="C"/>
+</segment>
+</net>
+<net name="N$2" class="0">
+<segment>
+<pinref part="R2" gate="G$1" pin="2"/>
+<pinref part="LED2" gate="G$1" pin="C"/>
+</segment>
+</net>
+<net name="N$3" class="0">
+<segment>
+<pinref part="R3" gate="G$1" pin="2"/>
+<pinref part="LED3" gate="G$1" pin="C"/>
+</segment>
+</net>
+<net name="N$4" class="0">
+<segment>
+<pinref part="R4" gate="G$1" pin="2"/>
+<pinref part="LED4" gate="G$1" pin="C"/>
+</segment>
+</net>

Commit message: v02 software + updated general hardware
Changed lines of the file:
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@@
 <part name="GND3" library="SparkFun-PowerSymbols" deviceset="GND" device=""/>
 <part name="GND4" library="SparkFun-PowerSymbols" deviceset="GND" device=""/>
-<part name="GND6" library="SparkFun-PowerSymbols" deviceset="GND" device=""/>
 <part name="GND7" library="SparkFun-PowerSymbols" deviceset="GND" device=""/>
-<part name="SUPPLY1" library="SparkFun-PowerSymbols" deviceset="VCC" device=""/>
 <part name="SUPPLY2" library="SparkFun-PowerSymbols" deviceset="VCC" device=""/>
 <part name="GND8" library="supply1" library_urn="urn:adsk.eagle:library:371" deviceset="GND" device=""/>
@@
 <instance part="GND3" gate="1" x="198.12" y="83.82" rot="R180"/>
 <instance part="GND4" gate="1" x="205.74" y="83.82" rot="R180"/>
-<instance part="GND6" gate="1" x="132.08" y="15.24" rot="R180"/>
 <instance part="GND7" gate="1" x="0" y="81.28" rot="R180"/>
-<instance part="SUPPLY1" gate="G$1" x="124.46" y="12.7"/>
 <instance part="SUPPLY2" gate="G$1" x="0" y="96.52"/>
 <instance part="GND8" gate="1" x="58.42" y="30.48"/>
